File: FT232HQ-FIFO.kicad_pcb (KiCad board)
At the start: 2 copper layers, 30.5 x 25.4 mm, 30 parts, among them J1 USB_C_Receptacle_USB2.0_16P, J2 Conn_02x10_Odd_Even, U2 TLV75533PDBV, U4 12M, U5 FT232H, U6 93LCxxBxxOT

Commit message: update
Parts:
- J2: footprint 1st_commonly:DC3_02x10_2.54_Odd_Even -> Connector_PinHeader_2.54mm:PinHeader_2x10_P2.54mm_Vertical
- moved J2 11.6 mm to (149.8, 87.4)
- moved C13 2.62 mm to (141.9, 79.8), turned to 90 degrees
- moved R5 0.15 mm to (141.9, 73.2)
Connections:
- J2 pad 19: /AC8 -> GND
- J2 pad 20: /AC9 -> GND
Routing:
- net /AC9: track 14.8 -> 0.00 mm, vias 1 -> 0
- net /AC8: track 13.8 -> 0.00 mm
- net /AD0: track 16.3 -> 19.3 mm
- net GND: track 9.11 -> 6.34 mm
- net /AC2: track 8.98 -> 11.7 mm
- net /AC6: track 12.2 -> 14.8 mm
- net /AC4: track 10.6 -> 13.2 mm
- net /AD2: track 14.9 -> 17.3 mm
- net /AC0: track 13.3 -> 15.6 mm
- net /AD6: track 13.4 -> 15.5 mm
- net /AD4: track 14.0 -> 16.0 mm
- net /AD3: track 15.1 -> 13.2 mm, vias 1 -> 0
- net /AD5: track 14.4 -> 12.7 mm, vias 1 -> 0
- net /AD7: track 13.8 -> 12.2 mm, vias 1 -> 0
- net /AC3: track 10.5 -> 9.02 mm, vias 1 -> 0
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Other:
- board size 30.5 x 25.4 mm -> 31.8 x 25.4 mm
- board text removed: "AC8"
- board text removed: "AC9"
